File: jetson-orin-agx-baseboard.kicad_sch (KiCad schematic)
At the start: 0 parts

Commit message: [#81778] Add connector symbol
Other:
- added sheet SoM (SoM.kicad_sch)
Changed lines of the file:
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@@
 		(comment 1 "www.antmicro.com")
+	)
+	(sheet
+		(at 173.99 119.38)
+		(size 38.1 34.29)
+		(exclude_from_sim no)
+		(in_bom yes)
+		(on_board yes)
+		(dnp no)
+		(fields_autoplaced yes)
+		(stroke
+			(width 0.1524)
+			(type solid)
+		)
+		(fill
+			(color 0 0 0 0.0000)
+		)
+		(property "Sheetname" "SoM"
+			(at 173.99 118.6684 0)
+			(effects
+				(font
+					(size 1.27 1.27)
+				)
+				(justify left bottom)
+			)
+		)
+		(property "Sheetfile" "SoM.kicad_sch"
+			(at 173.99 154.2546 0)
+			(effects
+				(font
+					(size 1.27 1.27)
+				)
+				(justify left top)
+			)
+		)
+		(instances
+			(project "jetson-orin-agx-baseboard"
+				(path "/f569b0be-0afd-48b7-93ee-28582a4c645c"
+					(page "2")
+				)
+			)
+		)
 	)
 	(sheet_instances

Commit message: [#81970] Refactor root
Other:
- removed sheet SoM
- added sheet CSI (CSI.kicad_sch)
- added sheet Debug (Debug.kicad_sch)
- added sheet Ethernet (Ethernet.kicad_sch)
- added sheet Expansion connector (Expansion_connector.kicad_sch)
- added sheet HDMI (HDMI.kicad_sch)
- added sheet M.2 (m2.kicad_sch)
- added sheet OCuLink (Oculink.kicad_sch)
- added sheet Peripherals (Peripherals.kicad_sch)
- added sheet Power (Power.kicad_sch)
- added sheet SoM_IO (SoM_io.kicad_sch)
- added sheet SoM_IO2 (SoM_io2.kicad_sch)
- added sheet SoM_ctrl (SoM_ctrl.kicad_sch)
- added sheet SoM_debug (SoM_debug.kicad_sch)
- added sheet USB (USB.kicad_sch)
- added sheet USB Debug, DP (USB_debug_dp.kicad_sch)
- note added: "SoM"
