File: Ethernet.kicad_sch (KiCad schematic)
At the start: 0 parts

Commit message: [#81970] Add SFP sheet and power section
Parts:
- added C68: C_100n_100V_0805, antmicro-footprints:C_0805_2012Metric, symbol antmicroCapacitorsmisc:C_100n_100V_0805
- added C69: C_10n_0603, antmicro-footprints:C_0603_1608Metric, symbol antmicroCapacitors0603:C_10n_0603
- added C70, C72, C73, C74: C_22u_100V_2220, antmicro-footprints:C_2220_5650Metric, symbol antmicroCapacitorsmisc:C_22u_100V_2220
- added C71, C77: C_100n_0402, antmicro-footprints:C_0402_1005Metric, symbol antmicroCapacitors0402:C_100n_0402
- added C75, C76: C_47u_16V_1206, antmicro-footprints:C_1206_3216Metric, symbol antmicroCapacitorsmisc:C_47u_16V_1206
- added D11, D12: CD-MMBL110S, antmicro-footprints:DFN3538, symbol antmicroDiodesRectifiersSingle:CD-MMBL110S
- added D13: PTVS58VS1UR,115, antmicro-footprints:D_SOD-123F, symbol antmicroTVSDiodes:PTVS58VS1UR,115
- added D14: LED_G_0603_LTST-C190GKT, antmicro-footprints:LED_0603_1608Metric_G, symbol antmicroLEDIndicationDiscrete:LED_G_0603_LTST-C190GKT
- added FB1, FB2: FB_220Z_2A_Murata-BLM21PG_0805, antmicro-footprints:FB_0805_2012Metric, symbol antmicroFerriteBeadsandChips:FB_220Z_2A_Murata-BLM21PG_0805
- added J5: Bus_RJ45_5-2337992-8, antmicro-footprints:RJ45_X-2337992-8_Horizontal, symbol antmicroModularConnectorsJacksWithMagnetics:Bus_RJ45_5-2337992-8
- added Q6: PJE138K, antmicro-footprints:SOT-523, symbol antmicroTransistorsFETsMOSFETsSingle:PJE138K
- added R61: R_1k3_0402, antmicro-footprints:R_0402_1005Metric, symbol antmicroResistors0402:R_1k3_0402
- added R62: R_49k9_0402, antmicro-footprints:R_0402_1005Metric, symbol antmicroResistors0402:R_49k9_0402
- added R63, R75: R_0R_0402, antmicro-footprints:R_0402_1005Metric, symbol antmicroResistors0402:R_0R_0402
- added R64: R_63R4_0603, antmicro-footprints:R_0603_1608Metric, symbol antmicroResistors0603:R_63R4_0603
- added R65: R_1k2_0402, antmicro-footprints:R_0402_1005Metric, symbol antmicroResistors0402:R_1k2_0402
- added R66, R72: R_24k9_0402, antmicro-footprints:R_0402_1005Metric, symbol antmicroResistors0402:R_24k9_0402
- added R67, R68, R69, R70: R_10k_0402, antmicro-footprints:R_0402_1005Metric, symbol antmicroResistors0402:R_10k_0402
- added R71: R_200R_0402, antmicro-footprints:R_0402_1005Metric, symbol antmicroResistors0402:R_200R_0402
- added R73, R77: R_470k_0402, antmicro-footprints:R_0402_1005Metric, symbol antmicroResistors0402:R_470k_0402
- added R74, R78: R_100k_0402, antmicro-footprints:R_0402_1005Metric, symbol antmicroResistors0402:R_100k_0402
- added R76, R79: R_1k_0402, antmicro-footprints:R_0402_1005Metric, symbol antmicroResistors0402:R_1k_0402
- added R80, R81: R_0R_0603, antmicro-footprints:R_0603_1608Metric, symbol antmicroResistors0603:R_0R_0603
- added U10: TPS2372-4, antmicro-footprints:VQFN-20_5x5x1mm_P0.65mm, symbol antmicroPMICPowerDistributionSwitchesLoadDrivers:TPS2372-4
- added U11: ACPL-217-500E, antmicro-footprints:SOIC-4_4.55x2.6mm_P1.27mm, symbol antmicroOptoisolatorsLogicOutput:ACPL-217-500E
- added U12: ULS-12_8.3-D48N-C, antmicro-footprints:Conv_Murata_ULS-100W, symbol antmicroDCDCConverters:ULS-12_8.3-D48N-C
Connections:
- new net: D11.2, D12.2, FB1.1
- new net: R76.2, U11.3
- new net: R79.1, U11.2
- new net: D11.1, D12.1, FB2.1
- new net: C71.1, J5.19 (SHIELD), J5.20 (SHIELD), R71.2
- new net: D14.2 (A), R72.1
- new net: C69.2, J5.4 (P4), J5.5 (P5)
- new net: R80.2, R81.2, U12.6 (TRIM)
- new net +3V3: J5.15 (LED_GRN+), J5.17 (LED_YEL+)
- new net AMPS_CTL: R61.2, U10.8 (AMPS_CTL)
- new net CLSA: R64.2, U10.3 (CLSA)
- new net CLSB: R65.2, U10.6 (CLSB)
- new net DEN: R66.1, U10.2 (DEN)
- new net DISABLE_POE_DCDC: U11.1
- new net GND: C69.1, C71.2, C75.1, C76.1, C77.2, R71.1, R79.2, R81.1, U12.4 (VOUT-), U12.5 (SENSE-)
- new net GNDD: C70.1, C72.1, C73.1, C74.1, D14.1 (C), Q6.2 (S), R74.1, R76.1, R78.1, U10.11 (RTNA), U10.12 (RTNB), U12.3 (VIN-)
- new net MPS_DUTY: R63.1, U10.9 (MPS_DUTY)
- new net PAIR_12: D11.3, J5.11 (VC1)
- new net PAIR_36: D11.4, J5.12 (VC2)
- new net PAIR_78: D12.4, J5.13 (VC3)
- new net PAIR_910: D12.3, J5.14 (VC4)
- new net PG: R68.2, U10.13 (PG)
- new net POE: C75.2, C76.2, C77.1, R80.1, U12.7 (SENSE+), U12.8 (VOUT+)
- new net POE_ACTIVE: Q6.1 (G), R68.1, R73.1, R74.2, R75.2, U11.4
- new net REF: R62.2, U10.7 (REF)
- new net TPH: R67.1, U10.18 (TPH)
- new net TPL: R69.1, U10.17 (TPL)
- new net ULS-12_CTRL: Q6.3 (D), R75.1, R77.1, R78.2, U12.2 (CTRL)
- new net VDD: C68.2, C70.2, C72.2, C73.2, C74.2, D13.1 (C), FB1.2, R66.2, R67.2, R69.2, R70.2, R72.2, R73.2, R77.2, U10.1 (VDD), U12.1 (VIN+)
- new net VSS: C68.1, D13.2 (A), FB2.2, R61.1, R62.1, R63.2, R64.1, R65.1, U10.21 (PAD_VSSC), U10.4 (VSSA), U10.5 (VSSB)
- new net ~{BT}: R70.1, U10.19 (~{BT})
- no-connect marks 0 -> 2
Other:
- note added: "1/5.7 divider"
- note added: "Alternative MPNs: 6-2337992-8, TMJG4926HENL"
- note added: "Ethernet Connector"
- note added: "Power over Ethernet"

Commit message: [#81970] Route traces from root schematic on other schematics
Parts:
- removed C68: C_100n_100V_0805, antmicro-footprints:C_0805_2012Metric, symbol antmicroCapacitorsmisc:C_100n_100V_0805
- removed C69: C_10n_0603, antmicro-footprints:C_0603_1608Metric, symbol antmicroCapacitors0603:C_10n_0603
- removed C70, C72, C73, C74: C_22u_100V_2220, antmicro-footprints:C_2220_5650Metric, symbol antmicroCapacitorsmisc:C_22u_100V_2220
- removed C71, C77: C_100n_0402, antmicro-footprints:C_0402_1005Metric, symbol antmicroCapacitors0402:C_100n_0402
- removed C75, C76: C_47u_16V_1206, antmicro-footprints:C_1206_3216Metric, symbol antmicroCapacitorsmisc:C_47u_16V_1206
- removed D11, D12: CD-MMBL110S, antmicro-footprints:DFN3538, symbol antmicroDiodesRectifiersSingle:CD-MMBL110S
- removed D13: PTVS58VS1UR,115, antmicro-footprints:D_SOD-123F, symbol antmicroTVSDiodes:PTVS58VS1UR,115
- removed D14: LED_G_0603_LTST-C190GKT, antmicro-footprints:LED_0603_1608Metric_G, symbol antmicroLEDIndicationDiscrete:LED_G_0603_LTST-C190GKT
- removed FB1, FB2: FB_220Z_2A_Murata-BLM21PG_0805, antmicro-footprints:FB_0805_2012Metric, symbol antmicroFerriteBeadsandChips:FB_220Z_2A_Murata-BLM21PG_0805
- removed J5: Bus_RJ45_5-2337992-8, antmicro-footprints:RJ45_X-2337992-8_Horizontal, symbol antmicroModularConnectorsJacksWithMagnetics:Bus_RJ45_5-2337992-8
- removed Q6: PJE138K, antmicro-footprints:SOT-523, symbol antmicroTransistorsFETsMOSFETsSingle:PJE138K
- removed R61: R_1k3_0402, antmicro-footprints:R_0402_1005Metric, symbol antmicroResistors0402:R_1k3_0402
- removed R62: R_49k9_0402, antmicro-footprints:R_0402_1005Metric, symbol antmicroResistors0402:R_49k9_0402
- removed R63, R75: R_0R_0402, antmicro-footprints:R_0402_1005Metric, symbol antmicroResistors0402:R_0R_0402
- removed R64: R_63R4_0603, antmicro-footprints:R_0603_1608Metric, symbol antmicroResistors0603:R_63R4_0603
- removed R65: R_1k2_0402, antmicro-footprints:R_0402_1005Metric, symbol antmicroResistors0402:R_1k2_0402
- removed R66, R72: R_24k9_0402, antmicro-footprints:R_0402_1005Metric, symbol antmicroResistors0402:R_24k9_0402
- removed R67, R68, R69, R70: R_10k_0402, antmicro-footprints:R_0402_1005Metric, symbol antmicroResistors0402:R_10k_0402
- removed R71: R_200R_0402, antmicro-footprints:R_0402_1005Metric, symbol antmicroResistors0402:R_200R_0402
- removed R73, R77: R_470k_0402, antmicro-footprints:R_0402_1005Metric, symbol antmicroResistors0402:R_470k_0402
- removed R74, R78: R_100k_0402, antmicro-footprints:R_0402_1005Metric, symbol antmicroResistors0402:R_100k_0402
- removed R76, R79: R_1k_0402, antmicro-footprints:R_0402_1005Metric, symbol antmicroResistors0402:R_1k_0402
- removed R80, R81: R_0R_0603, antmicro-footprints:R_0603_1608Metric, symbol antmicroResistors0603:R_0R_0603
- removed U10: TPS2372-4, antmicro-footprints:VQFN-20_5x5x1mm_P0.65mm, symbol antmicroPMICPowerDistributionSwitchesLoadDrivers:TPS2372-4
- removed U11: ACPL-217-500E, antmicro-footprints:SOIC-4_4.55x2.6mm_P1.27mm, symbol antmicroOptoisolatorsLogicOutput:ACPL-217-500E
- removed U12: ULS-12_8.3-D48N-C, antmicro-footprints:Conv_Murata_ULS-100W, symbol antmicroDCDCConverters:ULS-12_8.3-D48N-C
Connections:
- no-connect marks 2 -> 0
Other:
- note removed: "1/5.7 divider"
- note removed: "Alternative MPNs: 6-2337992-8, TMJG4926HENL"
- note removed: "Ethernet Connector"
- note removed: "Power over Ethernet"
