File: SoM_debug.kicad_sch (KiCad schematic)
At the start: 1 part, among them J2 Hermaphroditic_Molex_203456-0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

Commit message: [#81970] Refactor root
Parts:
- renumbered J2 to J1
Changed lines of the file:
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@@
 		(dnp no)
 		(fields_autoplaced yes)
-		(property "Reference" "J2"
+		(property "Reference" "J1"
 			(at 52.07 67.9449 0)
 			(effects
@@
 		(instances
 			(project "jetson-orin-agx-baseboard"
-				(path "/f569b0be-0afd-48b7-93ee-28582a4c645c/4579c4a7-22a6-485d-a5cb-a4d2e4f367db/9cc3f68f-dc6d-4cea-9df1-c11ad236ecf1"
-					(reference "J2")
+				(path "/f569b0be-0afd-48b7-93ee-28582a4c645c/58058c98-426b-4ff8-98ff-207367cfa3e6"
+					(reference "J1")
 					(unit 10)
 				)

Commit message: [#82757] Rename project to jetson-agx-thor-baseboard
Other:
- title: Jetson Orin AGX Baseboard -> Jetson AGX Thor Baseboard
Changed lines of the file:
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@@
 	(generator "eeschema")
 	(generator_version "9.0")
-	(paper "A4")
+	(paper "A3")
 	(title_block
-		(title "Jetson Orin AGX Baseboard")
+		(title "Jetson AGX Thor Baseboard")
 		(date "2025-08-11")
 		(rev "1.0.0")
