File: Power.kicad_sch (KiCad schematic)
At the start: 149 parts, among them J2 Molex_Nano-Fit_1x2_SMD_105430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, Q1 PJE138K, Q10 SQS401EN-T1_BE3, Q11 PJE138K, Q12 PJE138K, Q13 SQS401EN-T1_BE3, Q14 PJE138K, Q2 SQS401EN-T1_BE3, Q3 SQS401EN-T1_BE3, Q4 PJE138K, Q5 SSM3J332R, Q6 PJE138K, Q7 PJE138K, Q8 PJE138K, Q9 SQS401EN-T1_BE3, SW1 SW_SPDT_PCM12SMTR, U1 UCD9081, U2 LTC4412IS6, U3 74LVC2G14_SOT457, U4 74LVC1G175_SOT457, U5 SIC431AED-T1-GE3, U6 SIC431AED-T1-GE3, U7 SIC431AED-T1-GE3, U8 NCP730BMT330_WSON

Commit message: [#81970] Finalize connecting SFP+ to SOM
[#82054] Update SoM pins definitions

[#82054] Continue work on I2C

[#82330] Clean up

[#81970] Add SFP sheet and power section

[#82330] Annotation and clean up
Parts:
- removed BT1: Battery_Holder_MS621FE-FL11E, antmicro-footprints:MS621FE-FL11E, symbol antmicroBatteryHoldersClipsContacts:Battery_Holder_MS621FE-FL11E
- removed C1: C_100n_16V_X7R_0402, antmicro-footprints:C_0402_1005Metric, symbol antmicroCapacitors0402:C_100n_16V_X7R_0402
- removed C10, C33, C34, C35, C8, C9: C_100n_0402, antmicro-footprints:C_0402_1005Metric, symbol antmicroCapacitors0402:C_100n_0402
- removed C13, C14, C15, C16: C_22u_25V_0805, antmicro-footprints:C_0805_2012Metric, symbol antmicroCapacitorsmisc:C_22u_25V_0805
- removed C2: C_10n_0603, antmicro-footprints:C_0603_1608Metric, symbol antmicroCapacitors0603:C_10n_0603
- removed C3: C_100n_50V_X8L_0402, antmicro-footprints:C_0402_1005Metric, symbol antmicroCapacitors0402:C_100n_50V_X8L_0402
- removed C4, C59, C7: C_10u_0402, antmicro-footprints:C_0402_1005Metric, symbol antmicroCapacitors0402:C_10u_0402
- removed C52: C_10u_25V_0603, antmicro-footprints:C_0603_1608Metric, symbol antmicroCapacitors0603:C_10u_25V_0603
- removed C6: C_1u_25V_0402, antmicro-footprints:C_0402_1005Metric, symbol antmicroCapacitors0402:C_1u_25V_0402
- removed D11, D3, D6: RB521S30T1G, antmicro-footprints:SOD-523, symbol antmicroDiodesRectifiersSingle:RB521S30T1G
- removed D12: ESD9X5.0ST5G, antmicro-footprints:SOD-923, symbol antmicroTVSDiodes:ESD9X5.0ST5G
- removed D2, D7: TPD1E0B04_XDFN-2, antmicro-footprints:XDFN-2_1x0.60mm, symbol antmicroTVSDiodes:TPD1E0B04_XDFN-2
- removed Q1, Q11, Q12, Q14, Q6, Q7, Q8: PJE138K, antmicro-footprints:SOT-523, symbol antmicroTransistorsFETsMOSFETsSingle:PJE138K
- removed Q13, Q9: SQS401EN-T1_BE3, antmicro-footprints:Vishay_PowerPAK_1212-8_Single, symbol antmicroTransistorsFETsMOSFETsSingle:SQS401EN-T1_BE3
- removed Q5: SSM3J332R, antmicro-footprints:SOT-23-3, symbol antmicroTransistorsFETsMOSFETsSingle:SSM3J332R
- removed R1, R10, R14, R15, R18, R20, R33, R37, R39, R52, R53, R55, R57, R58, R59, R6, R8: R_10k_0402, antmicro-footprints:R_0402_1005Metric, symbol antmicroResistors0402:R_10k_0402
- removed R11: R_4k7_0402, antmicro-footprints:R_0402_1005Metric, symbol antmicroResistors0402:R_4k7_0402
- removed R12, R22, R9: R_200k_0402, antmicro-footprints:R_0402_1005Metric, symbol antmicroResistors0402:R_200k_0402
- removed R13: R_0R_22.4A_0603, antmicro-footprints:R_0603_1608Metric, symbol antmicroResistors0603:R_0R_22.4A_0603
- removed R17: R_22k_0402, antmicro-footprints:R_0402_1005Metric, symbol antmicroResistors0402:R_22k_0402
- removed R2, R34, R35, R36, R5: R_100k_0402, antmicro-footprints:R_0402_1005Metric, symbol antmicroResistors0402:R_100k_0402
- removed R21: R_200R_0402, antmicro-footprints:R_0402_1005Metric, symbol antmicroResistors0402:R_200R_0402
- removed R23: R_0R_0402, antmicro-footprints:R_0402_1005Metric, symbol antmicroResistors0402:R_0R_0402
- removed R40, R45, R48: R_470R_0402, antmicro-footprints:R_0402_1005Metric, symbol antmicroResistors0402:R_470R_0402
- removed R54: R_2k2_0402, antmicro-footprints:R_0402_1005Metric, symbol antmicroResistors0402:R_2k2_0402
- removed R56: R_0R_0603, antmicro-footprints:R_0603_1608Metric, symbol antmicroResistors0603:R_0R_0603
- removed R7: R_1k_0402, antmicro-footprints:R_0402_1005Metric, symbol antmicroResistors0402:R_1k_0402
- removed S1, S2: SW_KMR211NGLFS_SMD, antmicro-footprints:SW_KMR211NGLFS_SMD, symbol antmicroPushbuttonSwitches:SW_KMR211NGLFS_SMD
- removed SW1: SW_SPDT_PCM12SMTR, antmicro-footprints:PCM12SMTR, symbol antmicroSlideSwitches:SW_SPDT_PCM12SMTR
- removed TP3, TP6: TP_0.75mm_SMD, antmicro-footprints:TP_SMD_0.75mm, symbol antmicroTestPoints:TP_0.75mm_SMD
- removed U1: UCD9081, antmicro-footprints:HVQFN-32-1EP_5x5mm_P0.5mm_EP3.6x3.6mm, symbol antmicroPMICPowerSequencers:UCD9081
- removed U3: 74LVC2G14_SOT457, antmicro-footprints:SOT-23-6, symbol antmicroLogicBuffersDriversReceiversTransceivers:74LVC2G14_SOT457
- removed U4: 74LVC1G175_SOT457, antmicro-footprints:SOT-23-6, symbol antmicroLogicGatesandInverters:74LVC1G175_SOT457
- removed U8: NCP730BMT330_WSON, antmicro-footprints:WSON-6-1EP_2x2mm_P0.65mm, symbol antmicroPMICVoltageRegulatorsLinear:NCP730BMT330_WSON
- added C1, C2: C_100n_50V_X8L_0402, antmicro-footprints:C_0402_1005Metric, symbol antmicroCapacitors0402:C_100n_50V_X8L_0402
- added C10, C7, C8, C9: C_22u_25V_0805, antmicro-footprints:C_0805_2012Metric, symbol antmicroCapacitorsmisc:C_22u_25V_0805
- added C13, C14, C15, C16, C6: C_100n_0402, antmicro-footprints:C_0402_1005Metric, symbol antmicroCapacitors0402:C_100n_0402
- added C3, C4: C_1u_25V_0402, antmicro-footprints:C_0402_1005Metric, symbol antmicroCapacitors0402:C_1u_25V_0402
- added D2: DF2S30FS_SOD, antmicro-footprints:SOD-923, symbol antmicroTVSDiodes:DF2S30FS_SOD
- added Q2, Q7: SQS401EN-T1_BE3, antmicro-footprints:Vishay_PowerPAK_1212-8_Single, symbol antmicroTransistorsFETsMOSFETsSingle:SQS401EN-T1_BE3
- added Q8: SSM3K15ACT, antmicro-footprints:CST3-3, symbol antmicroTransistorsFETsMOSFETsSingle:SSM3K15ACT
- added R1: R_4k7_0402, antmicro-footprints:R_0402_1005Metric, symbol antmicroResistors0402:R_4k7_0402
- added R13: R_20k_0402, antmicro-footprints:R_0402_1005Metric, symbol antmicroResistors0402:R_20k_0402
- added R14: R_2k7_0402, antmicro-footprints:R_0402_1005Metric, symbol antmicroResistors0402:R_2k7_0402
- added R18: R_562k_0402, antmicro-footprints:R_0402_1005Metric, symbol antmicroResistors0402:R_562k_0402
- added R19: R_270k_0402, antmicro-footprints:R_0402_1005Metric, symbol antmicroResistors0402:R_270k_0402
- added R2, R33: R_0R_22.4A_0603, antmicro-footprints:R_0603_1608Metric, symbol antmicroResistors0603:R_0R_22.4A_0603
- added R20: R_39k_0402, antmicro-footprints:R_0402_1005Metric, symbol antmicroResistors0402:R_39k_0402
- added R21: R_0R_0402, antmicro-footprints:R_0402_1005Metric, symbol antmicroResistors0402:R_0R_0402
- added R32: R_10k_0402, antmicro-footprints:R_0402_1005Metric, symbol antmicroResistors0402:R_10k_0402
- added R82: R_1M_0402, antmicro-footprints:R_0402_1005Metric, symbol antmicroResistors0402:R_1M_0402
- added R83: R_100k_0201, antmicro-footprints:R_0201, symbol antmicroResistorsmisc:R_100k_0201
- added U2: LTC4412IS6, antmicro-footprints:SOT-23-6, symbol antmicroPMICORControllersIdealDiodes:LTC4412IS6
- R11: renamed from R28; now fitted
- R12: renamed from R29; now not fitted
- renumbered C37 to C33, C38 to C34, C39 to C35, C40 to C37, C41 to C38, C42 to C39, C43 to C40, C44 to C41, C45 to C42, C46 to C43, C47 to C44, C48 to C45, C49 to C46, C50 to C47, C51 to C48, C53 to C49, C54 to C50, C55 to C51, C56 to C52, C57 to C53, C58 to C54, D4 to D3, D5 to D4, D10 to D5, D8 to D6, D9 to D7, Q2 to Q1, Q10 to Q5, R27 to R10, R30 to R15, R31 to R16, R32 to R17, R38 to R22, R41 to R23, R42 to R24, R43 to R25, R44 to R26, R46 to R27, R47 to R28, R51 to R29, R49 to R30, R50 to R31, R16 to R5, R19 to R6, R24 to R7, R25 to R8, R26 to R9, TP4 to TP3, TP7 to TP4, U2 to U1, U5 to U3, U6 to U4, U7 to U5
Connections:
- net +3V3_AON is gone; now on net +3V3: D6.1 (C), R30.2, TP3.1
- net 3V3_STDB is gone; now on net +5V: TP5.1
- net +12V: now also D7.1 (C), R31.2, Q7.5 (D)
- net +3V3: now also R82.2
- net +5V: now also R33.2
- net 12V_EN: now also C36.1, Q7.4 (G), Q8.3 (D), R18.1, R19.2, R83.1; no longer U3.19 (EN), U4.19 (EN)
- net 5V_GATE: now also Q4.3 (D), R32.1
- net DC_IN: now also C1.2
- net GND: now also C36.2, C1.1, C10.1, C13.2, C14.2, C15.2, C16.2, C2.1, C3.1, C4.1, C7.1, C8.1, C9.1, D2.2 (A), Q8.2 (S), R14.1, R20.1, U2.2 (GND), U2.3 (CTL); no longer C36.1, C5.1
- net USBPD0_HV: now also C12.2, U5.1 (V_{IN}), U5.2 (V_{IN}), U5.22 (V_{IN}), U5.26 (V_{IN}), C15.1, C3.2, C4.2, C9.2, Q2.1 (S), Q2.2 (S), Q2.3 (S), R1.2, R2.1, U2.6 (SENSE)
- net VCC: now also C10.2, C13.1, C14.1, C6.2, C7.2, C8.2, R13.2, R18.2, R2.2; no longer C12.2, U5.1 (V_{IN}), U5.2 (V_{IN}), U5.22 (V_{IN}), U5.26 (V_{IN})
- net +5V_SoM: now reaches D5.1 (C), Q5.5 (D), R29.2
- net +5V_SoM: now also R32.2, R33.1
- net at Q3.4 (G), R5.2: now also C5.1, C6.1, R1.1
- net ~{RESET}: now reaches Q4.1 (G)
- net ~{RESET}: now also R21.1
- net 12V_OUT: no longer names the net of C45.2, C48.2, C51.2, C54.2, L3.2, R27.2, R31.1, U5.18 (V_{OUT})
- new net: Q2.4 (G), U2.5 (GATE)
- new net: R19.1, R20.2
- new net 3V3_EN: R21.2, U4.19 (EN)
- new net 5V_EN: C16.1, R13.1, R14.2, U3.19 (EN)
- new net POE: C2.2, D2.1 (C), Q2.5 (D), Q7.1 (S), Q7.2 (S), Q7.3 (S), R83.2, U2.1 (IN)
- new net PoE_STAT: Q8.1 (G), R82.1, U2.4 (STAT)
- no-connect marks 21 -> 7
Other:
- note removed: "12V @12A"
- note removed: "3.3V @150mA"
- note removed: "DISCHARGE CIRCUIT"
- note removed: "Ideal-diode O-Ring"
- note removed: "MODIFIED CIRCUIT FROM TI's SCEA048B AN"
- note removed: "NOTE: SW1 STARTUP CRTL 1-2 AUTO 3-2 MANUAL"
- note removed: "POWER BUTTON"
- note removed: "POWER-UP AND RESET CIRCUITRY"
- note removed: "Power sequencer"
- note removed: "RESET BUTTON"
- note removed: "RTC BACK-UP POWER"
- note removed: "SHORT PRESS - POWER UP LONG PRESS - POWER DOWN"
- note removed: "Soft start"
- note removed: "USB controller has an integrated ideal diode"
- note removed: "V_{OUT} = 0.6*(191k+10k)/10k = 12.06[V]"
- moved on the sheet: C33, C34, C35, C37, C38, C39, C40, C41, C42, C43, C44, C45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

Commit message: [#81782] Rebase power supply branch after review
Parts:
- removed C1, C2: C_100n_50V_X8L_0402, antmicro-footprints:C_0402_1005Metric, symbol antmicroCapacitors0402:C_100n_50V_X8L_0402
- removed C10, C7, C8, C9: C_22u_25V_0805, antmicro-footprints:C_0805_2012Metric, symbol antmicroCapacitorsmisc:C_22u_25V_0805
- removed C13, C14, C15, C16, C36, C6: C_100n_0402, antmicro-footprints:C_0402_1005Metric, symbol antmicroCapacitors0402:C_100n_0402
- removed C3, C4: C_1u_25V_0402, antmicro-footprints:C_0402_1005Metric, symbol antmicroCapacitors0402:C_1u_25V_0402
- removed D2, D4: DF2S30FS_SOD, antmicro-footprints:SOD-923, symbol antmicroTVSDiodes:DF2S30FS_SOD
- removed D7: ESD9X5.0ST5G, antmicro-footprints:SOD-923, symbol antmicroTVSDiodes:ESD9X5.0ST5G
- removed Q2, Q5, Q7: SQS401EN-T1_BE3, antmicro-footprints:Vishay_PowerPAK_1212-8_Single, symbol antmicroTransistorsFETsMOSFETsSingle:SQS401EN-T1_BE3
- removed Q8: SSM3K15ACT, antmicro-footprints:CST3-3, symbol antmicroTransistorsFETsMOSFETsSingle:SSM3K15ACT
- removed R1: R_4k7_0402, antmicro-footprints:R_0402_1005Metric, symbol antmicroResistors0402:R_4k7_0402
- removed R13: R_20k_0402, antmicro-footprints:R_0402_1005Metric, symbol antmicroResistors0402:R_20k_0402
- removed R14: R_2k7_0402, antmicro-footprints:R_0402_1005Metric, symbol antmicroResistors0402:R_2k7_0402
- removed R18: R_562k_0402, antmicro-footprints:R_0402_1005Metric, symbol antmicroResistors0402:R_562k_0402
- removed R19: R_270k_0402, antmicro-footprints:R_0402_1005Metric, symbol antmicroResistors0402:R_270k_0402
- removed R2, R33: R_0R_22.4A_0603, antmicro-footprints:R_0603_1608Metric, symbol antmicroResistors0603:R_0R_22.4A_0603
- removed R20: R_39k_0402, antmicro-footprints:R_0402_1005Metric, symbol antmicroResistors0402:R_39k_0402
- removed R21: R_0R_0402, antmicro-footprints:R_0402_1005Metric, symbol antmicroResistors0402:R_0R_0402
- removed R32: R_10k_0402, antmicro-footprints:R_0402_1005Metric, symbol antmicroResistors0402:R_10k_0402
- removed R82: R_1M_0402, antmicro-footprints:R_0402_1005Metric, symbol antmicroResistors0402:R_1M_0402
- removed R83: R_100k_0201, antmicro-footprints:R_0201, symbol antmicroResistorsmisc:R_100k_0201
- removed U2: LTC4412IS6, antmicro-footprints:SOT-23-6, symbol antmicroPMICORControllersIdealDiodes:LTC4412IS6
- added C1: C_100n_16V_X7R_0402, antmicro-footprints:C_0402_1005Metric, symbol antmicroCapacitors0402:C_100n_16V_X7R_0402
- added C101, C6, C98: C_1u_25V_0402, antmicro-footprints:C_0402_1005Metric, symbol antmicroCapacitors0402:C_1u_25V_0402
- added C102, C33, C34, C35, C4, C64, C65, C9, C97: C_100n_0402, antmicro-footprints:C_0402_1005Metric, symbol antmicroCapacitors0402:C_100n_0402
- added C13, C14, C15, C16: C_22u_25V_0805, antmicro-footprints:C_0805_2012Metric, symbol antmicroCapacitorsmisc:C_22u_25V_0805
- added C2: C_10n_0603, antmicro-footprints:C_0603_1608Metric, symbol antmicroCapacitors0603:C_10n_0603
- added C3: C_100n_50V_X8L_0402, antmicro-footprints:C_0402_1005Metric, symbol antmicroCapacitors0402:C_100n_50V_X8L_0402
- added C52: C_10u_25V_0603, antmicro-footprints:C_0603_1608Metric, symbol antmicroCapacitors0603:C_10u_25V_0603
- added C59, C62: C_10u_0402, antmicro-footprints:C_0402_1005Metric, symbol antmicroCapacitors0402:C_10u_0402
- added C61, C63: C_1u_0402, antmicro-footprints:C_0402_1005Metric, symbol antmicroCapacitors0402:C_1u_0402
- added D12, D14: ESD9X5.0ST5G, antmicro-footprints:SOD-923, symbol antmicroTVSDiodes:ESD9X5.0ST5G
- added D13: TPD1E0B04_XDFN-2, antmicro-footprints:XDFN-2_1x0.60mm, symbol antmicroTVSDiodes:TPD1E0B04_XDFN-2
- added D2, D3, D6, D7: LED_G_0603_LTST-C190GKT, antmicro-footprints:LED_0603_1608Metric_G, symbol antmicroLEDIndicationDiscrete:LED_G_0603_LTST-C190GKT
- added D35: BAT54C, antmicro-footprints:SOT-23-3, symbol antmicroDiodesRectifiersSingle:BAT54C
- added D5: SMF4L15A, antmicro-footprints:SOD-123FL, symbol antmicroTVSDiodes:SMF4L15A
- added Q1, Q7, Q8: PJE138K, antmicro-footprints:SOT-523, symbol antmicroTransistorsFETsMOSFETsSingle:PJE138K
- added Q10, Q11: BSS138-7-F, antmicro-footprints:SOT-23-3, symbol antmicroTransistorsFETsMOSFETsSingle:BSS138-7-F
- added Q12, Q5, Q6: IRLML6344TRPBF, antmicro-footprints:SOT-23-3, symbol antmicroTransistorsFETsMOSFETsSingle:IRLML6344TRPBF
- added R1, R10, R14, R15, R175, R18, R21, R22, R23, R33, R34, R35, R37, R39, R5, R55, R58, R7, R8: R_10k_0402, antmicro-footprints:R_0402_1005Metric, symbol antmicroResistors0402:R_10k_0402
- added R11: R_4k7_0402, antmicro-footprints:R_0402_1005Metric, symbol antmicroResistors0402:R_4k7_0402
- added R12, R20, R323, R6, R9: R_1k_0402, antmicro-footprints:R_0402_1005Metric, symbol antmicroResistors0402:R_1k_0402
- added R13: R_0R_22.4A_0603, antmicro-footprints:R_0603_1608Metric, symbol antmicroResistors0603:R_0R_22.4A_0603
- added R17: R_22k_0402, antmicro-footprints:R_0402_1005Metric, symbol antmicroResistors0402:R_22k_0402
- added R173, R2: R_100k_0402, antmicro-footprints:R_0402_1005Metric, symbol antmicroResistors0402:R_100k_0402
- added R174, R177: R_0R_0402, antmicro-footprints:R_0402_1005Metric, symbol antmicroResistors0402:R_0R_0402
- added R40, R45, R48: R_470R_0402, antmicro-footprints:R_0402_1005Metric, symbol antmicroResistors0402:R_470R_0402
- added R52: R_200k_0402, antmicro-footprints:R_0402_1005Metric, symbol antmicroResistors0402:R_200k_0402
- added R56, R63: R_0R_0603, antmicro-footprints:R_0603_1608Metric, symbol antmicroResistors0603:R_0R_0603
- added S4: SW_KMR211NGLFS_SMD, antmicro-footprints:SW_KMR211NGLFS_SMD, symbol antmicroPushbuttonSwitches:SW_KMR211NGLFS_SMD
- added SW2: SW_1-1825027-1_THT, antmicro-footprints:SW_1-1825027-1_THT, symbol antmicroPushbuttonSwitches:SW_1-1825027-1_THT
- added SW3: SW_SPDT_PCM12SMTR, antmicro-footprints:PCM12SMTR, symbol antmicroSlideSwitches:SW_SPDT_PCM12SMTR
- added TP4, TP6, TP8, TP9: TP_0.75mm_SMD, antmicro-footprints:TP_SMD_0.75mm, symbol antmicroTestPoints:TP_0.75mm_SMD
- added U1: UCD9081, antmicro-footprints:HVQFN-32-1EP_5x5mm_P0.5mm_EP3.6x3.6mm, symbol antmicroPMICPowerSequencers:UCD9081
- added U10: TPS7A0518P_SOT23-5, antmicro-footprints:SOT-23-5, symbol antmicroPMICVoltageRegulatorsLinear:TPS7A0518P_SOT23-5
- added U3: 74LVC1G00GM_115, antmicro-footprints:XSON-6_1x1.45mm_P0.5mm, symbol antmicroLogicGatesandInverters:74LVC1G00GM_115
- added U32: TPS3840PL30DBVR, antmicro-footprints:SOT-23-5, symbol antmicroPMICPowerSequencers:TPS3840PL30DBVR
- added U34: LTC2950CTS8-1, antmicro-footprints:SOT-23-8, symbol antmicroPMICPowerSequencers:LTC2950CTS8-1
- added U8: NCP730BMT330_WSON, antmicro-footprints:WSON-6-1EP_2x2mm_P0.65mm, symbol antmicroPMICVoltageRegulatorsLinear:NCP730BMT330_WSON
- R28: renamed from R11; now not fitted
- R29: renamed from R12; now fitted
- renumbered C33 to C37, C34 to C38, C35 to C39, C37 to C40, C38 to C41, C39 to C42, C40 to C43, C41 to C44, C42 to C45, C43 to C46, C44 to C47, C45 to C48, C46 to C49, C47 to C50, C48 to C51, C49 to C53, C50 to C54, C51 to C55, C52 to C56, C53 to C57, C54 to C58, D5 to D10, D3 to D4, D6 to D8, Q1 to Q2, R5 to R16, R6 to R19, R7 to R24, R8 to R25, R9 to R26, R10 to R27, R15 to R30, R16 to R31, R17 to R32, R22 to R38, R23 to R41, R24 to R42, R25 to R43, R26 to R44, R27 to R46, R28 to R47, R30 to R49, R31 to R50, R29 to R51, TP4 to TP7, U1 to U2, U3 to U5, U4 to U6, U5 to U7
Connections:
- net +12V: now also R45.2; no longer R50.2, TP7.1
- net +3V3: now also R48.2, R9.2, TP9.1, U1.6 (MON1); no longer TP3.1
- net +5V: now also R40.2; no longer TP5.1
- net +5V_SoM: now also C62.1, R12.2, R14.2, R20.2, TP6.1, U10.1 (VIN), U10.3 (EN)
- net DC_IN: now also C3.2
- net GND: now also C5.1, C1.1, C102.1, C13.1, C14.1, C15.1, C16.1, C2.1, C3.1, C33.2, C34.2, C35.2, C4.1, C52.1, C59.1, C61.1, C62.2, C63.1, C64.1, C65.1, C97.1, C98.1, D12.2 (A), D13.1 (C), D14.2 (A), D2.1 (C), D3.1 (C), D5.2 (A), D6.1 (C), Q1.2 (S), Q10.2 (S), Q11.2 (S), Q12.2 (S), Q5.2 (S), Q6.2 (S), Q7.2 (S), Q8.2 (S), R10.1, R15.1, R18.1, R21.1, R33.1, R34.1, R35.1, R37.1, R52.1, R55.1, R8.1, SW2.2, SW2.SH, SW3.S1 (SH), SW3.S2 (SH), SW3.S3 (SH), SW3.S4 (SH), U1.1 (GND), U1.29 (TEST), U1.33 (PAD), U10.2 (GND), U3.3 (GND), U32.3 (GND), U34.4 (GND), U8.3 (GND), U8.5 (PG), U8.7 (GND)
- net USBPD0_HV: now also Q3.1 (S), Q3.2 (S), Q3.3 (S), C6.2, R11.2, R13.1; no longer C12.2, Q3.5 (D), U7.1 (V_{IN}), U7.2 (V_{IN}), U7.22 (V_{IN}), U7.26 (V_{IN})
- net VCC: now also C12.2, Q3.5 (D), U7.1 (V_{IN}), U7.2 (V_{IN}), U7.22 (V_{IN}), U7.26 (V_{IN}), C13.2, C14.2, C15.2, C16.2, C33.1, C34.1, C35.1, C52.2, C9.2, R13.2, U8.4 (EN), U8.6 (V_{IN}); no longer Q3.1 (S), Q3.2 (S), Q3.3 (S)
- net at Q3.4 (G), R16.2: now also C6.1, C9.1, R11.1; no longer C5.1
- net 12V_OUT: now reaches C48.2, C51.2, C55.2, C58.2, L3.2, R46.2, R50.1, U7.18 (V_{OUT})
- net 12V_EN renamed SYS_VIN_HV_EN
- net SYS_VIN_HV_EN: now also R33.2, U1.11 (EN3)
- net 3V3_EN renamed SYS_VIN_SV_EN
- net SYS_VIN_SV_EN: now also R35.2, U1.23 (EN1)
- net 5V_EN renamed SYS_VIN_MV_EN
- net SYS_VIN_MV_EN: now also R34.2, U1.24 (EN2)
- net 5V_GATE: no longer names the net of Q4.3 (D)
- net 5V_GATE: now also R7.2, U3.2 (A)
- net ~{RESET} renamed ~{MODULE_SHDN_N}
- new net: Q12.1 (G), Q5.1 (G), Q6.1 (G), Q7.3 (D), R39.1
- new net: D2.2 (A), R12.1
- new net: R55.2, SW3.3
- new net: Q1.1 (G), R5.1, U1.10 (EN4)
- new net: R2.1, U1.32 (ROSC)
- new net: R14.1, R15.2, U1.7 (MON2)
- new net: R17.1, R18.2, U1.8 (MON3)
- new net: Q6.3 (D), R48.1
- new net: R174.1, R175.1, U34.8 (~{KILL})
- new net: D6.2 (A), R6.1
- new net: C98.2, U32.5 (CT)
- new net: Q5.3 (D), R45.1
- new net: R1.2, R323.2, U34.6 (EN)
- new net: D7.1 (C), Q8.3 (D)
- new net: D7.2 (A), R20.1
- new net: C65.2, D13.2 (A), Q10.1 (G), R52.2, S4.3, S4.4
- new net: SW3.2, U32.4 (~{MR})
- new net: C64.2, U34.3 (ONT)
- new net: R177.1, U34.5 (~{INT})
- new net: C61.2, U34.7 (OFFT)
- new net: Q12.3 (D), R40.1
- new net: D3.2 (A), R9.1
- new net: R174.2, U3.4 (Y)
- new net: Q11.1 (G), U32.1 (~{RESET})
- new net: C101.1, Q11.3 (D), R173.1
- new net +1V8: D14.1 (C), Q8.1 (G), R21.2, R63.2, TP8.1
- new net +3V3_STDB: C1.2, C102.2, C4.2, C97.2, D12.1 (C), D35.3, R1.1, R175.2, R2.2, R22.2, R23.2, R39.2, R5.2, R56.2, R58.1, R7.1, S4.1, S4.2, TP5.1, U1.3 (XIN), U1.30 (VCC), U3.6 (VCC), U32.2 (VDD), U34.1 (V_{IN})
- new net 1V8_LDO: C63.2, R63.1, U10.5 (VOUT)
- new net 3V3_LDO: C59.2, R56.1, U8.1 (V_{OUT})
- new net CARRIER_POWER_ON: R10.2, U1.9 (MON6)
- new net MODULE_POWER_ON: Q7.1 (G), R37.2, R8.2, U1.12 (EN5), U1.19 (MON5), U3.1 (B)
- new net PWRBTN: C101.2, D35.1, D35.2, R173.2, R58.2, SW2.1, U34.2 (~{PB})
- new net SYS_RESET_N: Q10.3 (D)
- new net SYS_SCL: R22.1, TP3.1, U1.22 (SCL)
- new net SYS_SDA: R23.1, TP4.1, U1.21 (SDA)
- new net VDDIN_PWR_BAD_N: Q1.3 (D), U1.18 (MON4)
- new net VDD_SoM_HV: D5.1 (C), R17.2, R50.2, R6.2, TP7.1
- new net ~{CW_PWRBTN}: R177.2
- new net ~{PWR_SEQ_RST}: C2.2, R323.1, U1.5 (~{RST})
- no-connect marks 7 -> 20
Other:
- note added: "12V @12A"
- note added: "1V8 LDO"
- note added: "3-2 manual 1-2 auto"
- note added: "3.3V @150mA"
- note added: "3V3 STANDBY LDO"
- note added: "DISCHARGE CIRCUIT"
- note added: "Ideal-diode O-Ring"
- note added: "Power button"
- note added: "Power sequencer"
- note added: "Power-up and reset"
- note added: "Reset button"
- note added: "Simulate button click for autostart"
- note added: "Soft start"
- note added: "USB controller has an integrated ideal diode"
- note added: "V_{OUT} = 0.6*(191k+10k)/10k = 12.06[V]"
- moved on the sheet: C37, C38, C39, C40, C41, C42, C43, C44, C45, C46, C47, C48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

Commit message: [#82757] Rename project to jetson-agx-thor-baseboard
Other:
- title: Jetson Orin AGX Baseboard -> Jetson AGX Thor Baseboard
Changed lines of the file:
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@@
 	(paper "A3")
 	(title_block
-		(title "Jetson Orin AGX Baseboard")
+		(title "Jetson AGX Thor Baseboard")
 		(date "2025-08-11")
 		(rev "1.0.0")

Commit message: [#82757] Cleanup: reorganise page numbers and fix annotations
Parts:
- renumbered C2 to C28, C1 to C29, C3 to C30, C4 to C31, C97 to C32, C98 to C33, C5 to C34, C101 to C35, C6 to C36, C102 to C37, C9 to C38, C65 to C39, C61 to C40, C64 to C41, C11 to C42, C12 to C43, C13 to C44, C14 to C45, C15 to C46, C16 to C47, C33 to C48, C34 to C49, C35 to C50, C62 to C51, C37 to C52, C38 to C53, C39 to C54, C40 to C55, C41 to C56, C42 to C57, C63 to C58, C43 to C59, C44 to C60, C45 to C61, C52 to C62, C46 to C63, C47 to C64, C48 to C65, C49 to C66, C50 to C67, C51 to C68, C53 to C69, C54 to C70, C55 to C71, C56 to C72, C57 to C73, C58 to C74, C59 to C75, D5 to D10, D12 to D11, D2 to D12, D3 to D13, D6 to D14, D1 to D2, D35 to D3, D13 to D5, D14 to D6, D10 to D8, D8 to D9, Q4 to Q1, Q5 to Q10, Q6 to Q11, Q11 to Q3, Q3 to Q4, Q1 to Q5, Q10 to Q6, Q12 to Q8, Q8 to Q9, R7 to R10, R55 to R11, R23 to R12, R2 to R13, R58 to R14, R173 to R15, R11 to R16, R8 to R17, R10 to R18, R33 to R19, R13 to R20, R16 to R21, R34 to R22, R174 to R23, R35 to R24, R175 to R25, R52 to R26, R19 to R27, R5 to R28, R14 to R29, R15 to R30, R1 to R31, R177 to R32, R17 to R33, R18 to R34, R323 to R35, R24 to R36, R25 to R37, R26 to R38, R27 to R39, R28 to R40, R29 to R41, R30 to R42, R31 to R43, R32 to R44, R37 to R45, R63 to R46, R39 to R47, R38 to R48, R40 to R49, R21 to R50, R20 to R51, R41 to R52, R42 to R53, R43 to R54, R44 to R55, R45 to R56, R46 to R57, R47 to R58, R48 to R59, R51 to R60, R49 to R61, R50 to R62, R56 to R63, R12 to R64, R9 to R65, R6 to R66, R22 to R9, S4 to S1, SW3 to SW1, TP3 to TP1, TP4 to TP2, TP1 to TP3, TP2 to TP4, TP8 to TP5, TP9 to TP6, TP6 to TP7, TP7 to TP8, TP5 to TP9, U34 to U10, U10 to U11, U5 to U12, U6 to U13, U7 to U14, U8 to U15, U2 to U6, U3 to U7, U1 to U8, U32 to U9
