File: USB.kicad_sch (KiCad schematic)
At the start: 87 parts, among them J1 PinHeader_1x3_P2.54mm_Drill1.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, J2 USB-C_Amphenol_12401598E4, J3 USB-C_Amphenol_12401598E4, J4 USB-C_Amphenol_12401598E4, U1 HD3SS3220IRNHR, U10 TPD4E05U06QDQARQ1, U2 AP7366_SOT, U3 TPD4E05U06QDQARQ1, U4 TPD4E05U06QDQARQ1, U5 USB7252C, U52 TPD4E05U06QDQARQ1, U53 TPD4E05U06QDQARQ1, U54 TPD4E05U06QDQARQ1, U6 W25Q80DV_USON, U7 TPD4E05U06QDQARQ1, U8 TPD4E05U06QDQARQ1, U9 TPD4E05U06QDQARQ1, Y1 Oscillator_25MHz_ESC_2016MV

Commit message: [#82757] Rename project to jetson-agx-thor-baseboard
Other:
- title: Jetson Orin AGX Baseboard -> Jetson AGX Thor Baseboard
Changed lines of the file:
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@@
 	(paper "A3")
 	(title_block
-		(title "Jetson Orin AGX Baseboard")
+		(title "Jetson AGX Thor Baseboard")
 		(date "2025-08-11")
 		(rev "1.0.0")

Commit message: [#82757] Cleanup: reorganise page numbers and fix annotations
Parts:
- renumbered C25 to C100, C31 to C101, C32 to C102, C27 to C103, C28 to C104, C35 to C105, C36 to C106, C29 to C107, C30 to C108, C37 to C109, C38 to C110, C26 to C111, C33 to C112, C34 to C113, C39 to C114, C40 to C115, C41 to C116, C42 to C117, C3 to C76, C1 to C77, C2 to C78, C9 to C79, C4 to C80, C5 to C81, C6 to C82, C7 to C83, C8 to C84, C10 to C85, C11 to C86, C12 to C87, C13 to C88, C14 to C89, C15 to C90, C16 to C91, C17 to C92, C18 to C93, C19 to C94, C20 to C95, C21 to C96, C22 to C97, C23 to C98, C24 to C99, D1 to D15, J1 to J3, J2 to J4, J4 to J5, J3 to J6, R4 to R67, R1 to R68, R2 to R69, R3 to R70, R7 to R71, R8 to R72, R5 to R73, R6 to R74, R9 to R75, R10 to R76, R11 to R77, R13 to R78, R12 to R79, R14 to R80, R15 to R81, R16 to R82, R17 to R83, R18 to R84, R19 to R85, R20 to R86, R21 to R87, R22 to R88, R23 to R89, R24 to R90, R25 to R91, R26 to R92, U2 to U16, U1 to U17, U3 to U18, U52 to U19, U4 to U20, U5 to U21, U6 to U22, U7 to U23, U8 to U24, U53 to U25, U10 to U26, U9 to U27, U54 to U28, Y1 to Y2
