File: som_io2.kicad_sch (KiCad schematic)
At the start: 8 parts, among them J1 Hermaphroditic_Molex_203456-0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, Y1 Oscillator_156.25MHz_SG3225EEN

Commit message: [#82837] Swap SoM form AGX Orin to Thor with all of its connections
Parts:
- removed J1: Hermaphroditic_Molex_203456-0003_CUSTOM_Jetson_Or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, antmicro-footprints:Conn_Hermaphroditic_Molex_203456-0003_mirrored, symbol antmicroB2BConnectors:Hermaphroditic_Molex_203456-0003_CUSTOM_Jetson_Orin_AGX_H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
- added C237, C238: C_100n_50V_X8L_0402, antmicro-footprints:C_0402_1005Metric, symbol antmicroCapacitors0402:C_100n_50V_X8L_0402
- added J1: Hermaphroditic_Molex_203456-0003_CUSTOM_Jetson_AG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, antmicro-footprints:Conn_Hermaphroditic_Molex_203456-0003_mirrored, symbol antmicroB2BConnectors:Hermaphroditic_Molex_203456-0003_CUSTOM_Jetson_AGX_Thor_H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
- added J20: Tag-Connect_TC2050-IDC-NL_2x5_P1.27mm, antmicro-footprints:Tag-Connect_TC2050-IDC-NL_2x5_P1.27mm, symbol antmicroTestPoints:Tag-Connect_TC2050-IDC-NL_2x5_P1.27mm
- added Q28: PJE138K, antmicro-footprints:SOT-523, symbol antmicroTransistorsFETsMOSFETsSingle:PJE138K
- added R126: R_100k_0402, antmicro-footprints:R_0402_1005Metric, symbol antmicroResistors0402:R_100k_0402
- added R285: R_10k_0402, antmicro-footprints:R_0402_1005Metric, symbol antmicroResistors0402:R_10k_0402
- added R290, R291, R292, R293, R294, R295: R_0R_0402, antmicro-footprints:R_0402_1005Metric, symbol antmicroResistors0402:R_0R_0402
- added U59: TXU0304BQAR, antmicro-footprints:DHVQFN-14-1EP_2.5x3mm, symbol antmicroLogicTranslatorsLevelShifters:TXU0304BQAR
Connections:
- net CSI0.CLK+: now also J1.F43 (CSI0_CLK_P)
- net CSI0.CLK-: now also J1.F42 (CSI0_CLK_N)
- net CSI0.D0+: now also J1.E42 (CSI0_D0_P)
- net CSI0.D0-: now also J1.E41 (CSI0_D0_N)
- net CSI0.D1+: now also J1.E39 (CSI0_D1_P)
- net CSI0.D1-: now also J1.E38 (CSI0_D1_N)
- net CSI0.D2+: now also J1.G41 (CSI1_D0_P)
- net CSI0.D2-: now also J1.G42 (CSI1_D0_N)
- net CSI0.D3+: now also J1.J41 (CSI1_D1_P)
- net CSI0.D3-: now also J1.J42 (CSI1_D1_N)
- net CSI1.CLK+: now also J1.B43 (CSI2_CLK_P)
- net CSI1.CLK-: now also J1.B42 (CSI2_CLK_N)
- net CSI1.D0+: now also J1.A41 (CSI2_D0_P)
- net CSI1.D0-: now also J1.A42 (CSI2_D0_N)
- net CSI1.D1+: now also J1.C42 (CSI2_D1_P)
- net CSI1.D1-: now also J1.C41 (CSI2_D1_N)
- net CSI1.D2+: now also J1.E45 (CSI3_D0_P)
- net CSI1.D2-: now also J1.E44 (CSI3_D0_N)
- net CSI1.D3+: now also J1.G44 (CSI3_D1_P)
- net CSI1.D3-: now also J1.G45 (CSI3_D1_N)
- net CSI2.CLK+: now also J1.F48 (CSI4_CLK_P)
- net CSI2.CLK-: now also J1.F49 (CSI4_CLK_N)
- net CSI2.D0+: now also J1.G48 (CSI4_D0_P)
- net CSI2.D0-: now also J1.G47 (CSI4_D0_N)
- net CSI2.D1+: now also J1.E47 (CSI4_D1_P)
- net CSI2.D1-: now also J1.E48 (CSI4_D1_N)
- net CSI2.D2+: now also J1.D42 (CSI5_D0_P)
- net CSI2.D2-: now also J1.D43 (CSI5_D0_N)
- net CSI2.D3+: now also J1.D46 (CSI5_D1_P)
- net CSI2.D3-: now also J1.D45 (CSI5_D1_N)
- net CSI3.CLK+: now also J1.J44 (CSI6_CLK_P)
- net CSI3.CLK-: now also J1.J45 (CSI6_CLK_N)
- net CSI3.D0+: now also J1.K44 (CSI6_D0_P)
- net CSI3.D0-: now also J1.K43 (CSI6_D0_N)
- net CSI3.D1+: now also J1.H46 (CSI6_D1_P)
- net CSI3.D1-: now also J1.H45 (CSI6_D1_N)
- net CSI3.D2+: now also J1.A44 (CSI7_D0_P)
- net CSI3.D2-: now also J1.A45 (CSI7_D0_N)
- net CSI3.D3+: now also J1.C47 (CSI7_D1_P)
- net CSI3.D3-: now also J1.C48 (CSI7_D1_N)
- net DP0.AUX+: now also J1.G53 (DP_AUX_CH0_P)
- net DP0.AUX-: now also J1.G54 (DP_AUX_CH0_N)
- net DP0.HPD: now also J1.K50 (HPD0)
- net DP0.TX0+: now also J1.D51 (DP0_D0_HDMI_D2_P)
- net DP0.TX0-: now also J1.D52 (DP0_D0_HDMI_D2_N)
- net DP0.TX1+: now also J1.B51 (DP0_D1_HDMI_D1_P)
- net DP0.TX1-: now also J1.B52 (DP0_D1_HDMI_D1_N)
- net DP0.TX2+: now also J1.A51 (DP0_D2_HDMI_D0_P)
- net DP0.TX2-: now also J1.A50 (DP0_D2_HDMI_D0_N)
- net DP0.TX3+: now also J1.C51 (DP0_D3_HDMI_CK_P)
- net DP0.TX3-: now also J1.C50 (DP0_D3_HDMI_CK_N)
- net DP1.AUX+: now also J1.D16 (DP_AUX_CH1_P)
- net DP1.AUX-: now also J1.D17 (DP_AUX_CH1_N)
- net DP1.HPD: now also J1.C18 (HPD1)
- net DP1.TX0+: now also J1.H49 (DP1_D0_HDMI_D2_P)
- net DP1.TX0-: now also J1.H48 (DP1_D0_HDMI_D2_N)
- net DP1.TX1+: now also J1.G51 (DP1_D1_HDMI_D1_P)
- net DP1.TX1-: now also J1.G50 (DP1_D1_HDMI_D1_N)
- net DP1.TX2+: now also J1.J47 (DP1_D2_HDMI_D0_P)
- net DP1.TX2-: now also J1.J48 (DP1_D2_HDMI_D0_N)
- net DP1.TX3+: now also J1.K46 (DP1_D3_HDMI_CK_P)
- net DP1.TX3-: now also J1.K47 (DP1_D3_HDMI_CK_N)
- net DP2.AUX+: now also J1.E19 (DP_AUX_CH2_P)
- net DP2.AUX-: now also J1.E18 (DP_AUX_CH2_N)
- net DP2.HPD: now also J1.A19 (HPD2)
- net DP2.TX0+: now also J1.A15 (DP2_D0_HDMI_D2_P)
- net DP2.TX0-: now also J1.A14 (DP2_D0_HDMI_D2_N)
- net DP2.TX1+: now also J1.J14 (DP2_D1_HDMI_D1_P)
- net DP2.TX1-: now also J1.J15 (DP2_D1_HDMI_D1_N)
- net DP2.TX2+: now also J1.C15 (DP2_D2_HDMI_D0_P)
- net DP2.TX2-: now also J1.C14 (DP2_D2_HDMI_D0_N)
- net DP2.TX3+: now also J1.G15 (DP2_D3_HDMI_CK_P)
- net DP2.TX3-: now also J1.G14 (DP2_D3_HDMI_CK_N)
- net DP3.AUX+: now also J1.F20 (DP_AUX_CH3_P)
- net DP3.AUX-: now also J1.F21 (DP_AUX_CH3_N)
- net DP3.HPD: now also J1.C19 (HPD3)
- net DP3.TX0+: now also J1.D33 (DP3_D0_HDMI_D2_P)
- net DP3.TX0-: now also J1.D32 (DP3_D0_HDMI_D2_N)
- net DP3.TX1+: now also J1.J35 (DP3_D1_HDMI_D1_P)
- net DP3.TX1-: now also J1.J34 (DP3_D1_HDMI_D1_N)
- net DP3.TX2+: now also J1.A34 (DP3_D2_HDMI_D0_P)
- net DP3.TX2-: now also J1.A35 (DP3_D2_HDMI_D0_N)
- net DP3.TX3+: now also J1.H32 (DP3_D3_HDMI_CK_P)
- net DP3.TX3-: now also J1.H33 (DP3_D3_HDMI_CK_N)
- net GND: now also C237.1, C238.1, J20.3, J20.5, J20.9, Q28.2 (S), R126.1, U59.15 (GND), U59.7 (GND)
- net PCIe_{C1x1}.RX0+: now also J1.B33 (UPHY_RX3_P)
- net PCIe_{C1x1}.RX0-: now also J1.B32 (UPHY_RX3_N)
- net PCIe_{C1x1}.TX0+: now also J1.G35 (UPHY_TX3_P)
- net PCIe_{C1x1}.TX0-: now also J1.G34 (UPHY_TX3_N)
- net PCIe_{C1x1}.~{CLKREQ}: now also J1.B37 (PEX_C1_CLKREQ_N)
- net PCIe_{C1x4}.~{RST}: now also J1.B36 (PEX_C1_RST_N)
- net PCIe_{C2x1}.RX0+: now also J1.D20 (UPHY_RX5_P)
- net PCIe_{C2x1}.RX0-: now also J1.D21 (UPHY_RX5_N)
- net PCIe_{C2x1}.TX0+: now also J1.H20 (UPHY_TX5_P)
- net PCIe_{C2x1}.TX0-: now also J1.H21 (UPHY_TX5_N)
- net PCIe_{C2x1}.~{CLKREQ}: now also J1.E11 (PEX_C2_CLKREQ_N)
- net PCIe_{C2x1}.~{RST}: now also J1.D10 (PEX_C2_RST_N)
- net PCIe_{C3x2}.CLK+: now also J1.F32 (UPHY_REFCLK3_P)
- net PCIe_{C3x2}.CLK-: now also J1.F33 (UPHY_REFCLK3_N)
- net PCIe_{C3x2}.RX0+: now also J1.B12 (UPHY_RX6_P)
- net PCIe_{C3x2}.RX0-: now also J1.B13 (UPHY_RX6_N)
- net PCIe_{C3x2}.RX1+: now also J1.D12 (UPHY_RX7_P)
- net PCIe_{C3x2}.RX1-: now also J1.D13 (UPHY_RX7_N)
- net PCIe_{C3x2}.TX0+: now also J1.K13 (UPHY_TX6_P)
- net PCIe_{C3x2}.TX0-: now also J1.K12 (UPHY_TX6_N)
- net PCIe_{C3x2}.TX1+: now also J1.H12 (UPHY_TX7_P)
- net PCIe_{C3x2}.TX1-: now also J1.H13 (UPHY_TX7_N)
- net PCIe_{C3x2}.~{CLKREQ}: now also J1.G8 (PEX_C3_CLKREQ_N)
- net PCIe_{C3x2}.~{RST}: now also J1.J9 (PEX_C3_RST_N)
- net PCIe_{C5x4}.CLK+: now also J1.E15 (UPHY_REFCLK5_P)
- net PCIe_{C5x4}.CLK-: now also J1.E14 (UPHY_REFCLK5_N)
- net PCIe_{C5x4}.RX0+: now also J1.D24 (UPHY_RX8_P)
- net PCIe_{C5x4}.RX0-: now also J1.D25 (UPHY_RX8_N)
- net PCIe_{C5x4}.RX1+: now also J1.B25 (UPHY_RX9_P)
- net PCIe_{C5x4}.RX1-: now also J1.B24 (UPHY_RX9_N)
- net PCIe_{C5x4}.RX2+: now also J1.C27 (UPHY_RX10_P)
- net PCIe_{C5x4}.RX2-: now also J1.C26 (UPHY_RX10_N)
- net PCIe_{C5x4}.RX3+: now also J1.A26 (UPHY_RX11_P)
- net PCIe_{C5x4}.RX3-: now also J1.A27 (UPHY_RX11_N)
- net PCIe_{C5x4}.TX0+: now also J1.H24 (UPHY_TX8_P)
- net PCIe_{C5x4}.TX0-: now also J1.H25 (UPHY_TX8_N)
- net PCIe_{C5x4}.TX1+: now also J1.K25 (UPHY_TX9_P)
- net PCIe_{C5x4}.TX1-: now also J1.K24 (UPHY_TX9_N)
- net PCIe_{C5x4}.TX2+: now also J1.G27 (UPHY_TX10_P)
- net PCIe_{C5x4}.TX2-: now also J1.G26 (UPHY_TX10_N)
- net PCIe_{C5x4}.TX3+: now also J1.J26 (UPHY_TX11_P)
- net PCIe_{C5x4}.TX3-: now also J1.J27 (UPHY_TX11_N)
- net PCIe_{C5x4}.~{CLKREQ}: now also J1.L19 (PEX_C5_CLKREQ_N)
- net PCIe_{C5x4}.~{RST}: now also J1.L18 (PEX_C5_RST_N)
- net SFI.RX+: now also J1.D28 (UPHY_RX12_P)
- net SFI.RX-: now also J1.D29 (UPHY_RX12_N)
- net SFI.TX+: now also J1.H28 (UPHY_TX12_P)
- net SFI.TX-: now also J1.H29 (UPHY_TX12_N)
- net USB0.D+: now also J1.F12 (USB0_P)
- net USB0.D-: now also J1.F13 (USB0_N)
- net USB1.D+: now also J1.C11 (USB1_P)
- net USB1.D-: now also J1.C10 (USB1_N)
- net USB2.D+: now also J1.A10 (USB2_P)
- net USB2.D-: now also J1.A11 (USB2_N)
- net USB3.D+: now also J1.G11 (USB3_P)
- net USB3.D-: now also J1.G10 (USB3_N)
- net USBSS0.RX+: now also J1.C34 (UPHY_RX0_P)
- net USBSS0.RX-: now also J1.C35 (UPHY_RX0_N)
- net USBSS0.TX+: now also J1.K32 (UPHY_TX0_P)
- net USBSS0.TX-: now also J1.K33 (UPHY_TX0_N)
- net USBSS1.RX+: now also J1.A22 (UPHY_RX1_P)
- net USBSS1.RX-: now also J1.A23 (UPHY_RX1_N)
- net USBSS1.TX+: now also J1.J22 (UPHY_TX1_P)
- net USBSS1.TX-: now also J1.J23 (UPHY_TX1_N)
- net USBSS2.RX+: now also J1.C23 (UPHY_RX2_P)
- net USBSS2.RX-: now also J1.C22 (UPHY_RX2_N)
- net USBSS2.TX+: now also J1.G23 (UPHY_TX2_P)
- net USBSS2.TX-: now also J1.G22 (UPHY_TX2_N)
- net ~{PEX_WAKE}: now also J1.A8 (PEX_WAKE_N)
- new net: C237.2, J20.1, U59.1 (VCCA)
- new net: R295.1, U59.10 (B4)
- new net: R292.1, U59.11 (B3Y)
- new net: R293.1, U59.12 (B2Y)
- new net: R294.1, U59.13 (B1Y)
- new net +1V8: C238.2, R285.2, R290.1, R291.1, U59.14 (VCCB), U59.8 (OE)
- new net JTAG_TCK: J1.A60 (JTAG_TCK), R292.2
- new net JTAG_TDI: J1.B60 (JTAG_TDI), R293.2
- new net JTAG_TDO: J1.D58 (JTAG_TDO), R295.2
- new net JTAG_TMS: J1.E58 (JTAG_TMS), R294.2
- new net JTAG_TRST_N: J1.G61 (JTAG_TRST_N), Q28.3 (D), R285.1
- new net NVDBG_SEL: J1.G60 (NVDBG_SEL), R291.2
- new net NVJTAG_SEL: J1.H59 (NVJTAG_SEL), R290.2
- new net PCIe_{C1x1}.CLK+: J1.F24 (UPHY_REFCLK1_P)
- new net PCIe_{C1x1}.CLK-: J1.F25 (UPHY_REFCLK1_N)
- new net PCIe_{C2x1}.CLK+: J1.F28 (UPHY_REFCLK2_P)
- new net PCIe_{C2x1}.CLK-: J1.F29 (UPHY_REFCLK2_N)
- new net TC_JTAG_TCK: J20.4, U59.4 (A3)
- new net TC_JTAG_TDI: J20.8, U59.3 (A2)
- new net TC_JTAG_TDO: J20.6, U59.5 (A4Y)
- new net TC_JTAG_TMS: J20.2, U59.2 (A1)
- new net TC_JTAG_TRST_N: J20.10, Q28.1 (G), R126.2
- no-connect marks 44 -> 54
Other:
- note added: "JTAG DEBUG"
- note removed: "Connect to ~{PEWAKE} pins on M.2"
